Commit message: "Past year of work"

File: src/prm_autobot_2023/urdf/robot_rm.urdf (robot description, URDF)
Before this commit: robot PRM_Autobot_2023, 3 links, 2 joints
Joints:
- joint base_link_joint: origin xyz=0.0 0.0 0.0 rpy=0 0 0 -> xyz=0.0 0.0 0.132 rpy=0 0 0
- joint lidar_joint: axis (none) -> 0 0 1; origin xyz=0.0 0.0 0.1 rpy=0 0 0 -> xyz=0.191 0.0 0.524 rpy=0 0 0; type fixed -> continuous

Commit message: Monday before comp - auto aim working on sentry verified

File: src/prm_autobot_2023/urdf/robot_rm.urdf (robot description, URDF)
Before this commit: robot PRM_Autobot_2023, 3 links, 2 joints
Joints:
- removed joint lidar_joint
